Commit message: Add files via upload

File: robot/urdf/robot.urdf (robot description, URDF)
Before this commit: robot robot, 6 links, 5 joints
Links:
- added link link5, mass 0.65092; collision mesh filename=package://robot/meshes/link5.STL; visual mesh filename=package://robot/meshes/link5.STL
Joints:
- added joint joint5: type revolute, parent link4, child link5, origin xyz=0 -0.075 0 rpy=0 0 0, axis -1 0 0, limit lower=0 upper=3.14 effort=100 velocity=3
- joint joint2: limit lower=-0.45 upper=-0 effort=200 velocity=0.1 -> lower=-0.41 upper=-0.015 effort=200 velocity=0.1
